File: MultiMifare.kicad_pcb (KiCad board)
At the start: 2 copper layers, 54 x 85.6 mm, 0 parts

Commit message: Misc
Parts:
- added SW1: SW_SPST, Button_Switch_SMD:SW_SPST_TL3342, F.Cu at (171.0, 134.5)
- added SW2: SW_SPST, Button_Switch_SMD:SW_SPST_TL3342, F.Cu at (157.0, 134.5)
- added U1: Mifare_Chip, MultiMifare:Mifare_Chip, F.Cu at (171.0, 120.0)
- added U2: Mifare_Chip, MultiMifare:Mifare_Chip, F.Cu at (157.0, 120.0)

Commit message: My first ugly KiCad project
Parts:
- added AE1: Antenna_Loop, MultiMifare:Mifare_Antenna, F.Cu at (152.1, 82.7)
Routing:
- net Net-(AE1-Pad1): track 0.00 -> 58.7 mm
- net Net-(AE1-Pad2): track 0.00 -> 43.7 mm, vias 0 -> 2
- net Net-(SW2-Pad1): track 0.00 -> 16.8 mm
- net Net-(SW1-Pad1): track 0.00 -> 10.5 mm
Changed lines of the file:
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@@
     (thickness 1.6)
     (drawings 8)
-    (tracks 0)
+    (tracks 17)
     (zones 0)
-    (modules 4)
+    (modules 5)
     (nets 5)
   )
@@
   )
   (setup
-    (last_trace_width 0.25)
+    (last_trace_width 0.762)
+    (user_trace_width 0.254)
+    (user_trace_width 0.508)
+    (user_trace_width 0.762)
+    (user_trace_width 1)
     (user_trace_width 1.5)
     (trace_clearance 0.2)
@@
     (add_net "Net-(SW2-Pad1)")
   )
+  (module MultiMifare:Mifare_Antenna (layer F.Cu)
+    (at 152.1 82.7 90)
+    (fp_text reference AE1 (at 0 0 90) (layer F.SilkS) hide
+      (effects (font (size 1.524 1.524) (thickness 0.3)))
+    )
+    (fp_text value Antenna_Loop (at 0 3 90) (layer F.SilkS) hide
+      (effects (font (size 1.524 1.524) (thickness 0.3)))
+    )
+    (fp_line (start -24.83 -24.807) (end -26.43 -24.807) (layer F.Cu) (width 0.391))
+    (fp_line (start -25.2 -25.2) (end -25.2 25.2) (layer B.CrtYd) (width 0.12))
+    (fp_line (start 25.2 25.2) (end -25.2 25.2) (layer B.CrtYd) (width 0.12))
+    (fp_line (start 25.2 -25.2) (end 25.2 25.2) (layer B.CrtYd) (width 0.12))
+    (fp_line (start -25.2 -25.2) (end 25.2 -25.2) (layer B.CrtYd) (width 0.12))
+    (fp_poly (pts (xy 25.005773 0.002645) (xy 25.003125 25.003125) (xy 0.002645 25.005773) (xy -24.997834 25.008421)
+      (xy -24.997834 -24.235834) (xy 24.246421 -24.235834) (xy 24.243773 0.002645) (xy 24.241125 24.241125)
+      (xy 0.002645 24.243773) (xy -24.235834 24.246421) (xy -24.235834 -23.473834) (xy 23.484421 -23.473834)
+      (xy 23.481773 0.002645) (xy 23.479125 23.479125) (xy 0.002645 23.481773) (xy -23.473834 23.484421)
+      (xy -23.473834 -22.711834) (xy 22.722421 -22.711834) (xy 22.719773 0.002645) (xy 22.717125 22.717125)
+      (xy 0.002645 22.719773) (xy -22.711834 22.722421) (xy -22.6905 -19.9) (xy -22.3095 -19.9)
+      (xy -22.330834 22.330833) (xy 22.330833 22.330833) (xy 22.330833 -22.341417) (xy -23.08225 -22.341417)
+      (xy -23.08225 23.092833) (xy 23.092833 23.092833) (xy 23.092833 -23.092834) (xy -23.84425 -23.092834)
+      (xy -23.84425 23.854833) (xy 23.854833 23.854833) (xy 23.854833 -23.854834) (xy -24.60625 -23.854834)
+      (xy -24.60625 24.616833) (xy 24.616833 24.616833) (xy 24.616833 -24.616834) (xy -24.997834 -24.616834)
+      (xy -24.997834 -24.997834) (xy 25.008421 -24.997834) (xy 25.005773 0.002645)) (layer F.Cu) (width 0.01))
+    (pad 1 smd rect (at -26.692 -24.81 90) (size 0.8 0.8) (layers F.Cu F.Paste F.Mask)
+      (net 3 "Net-(AE1-Pad1)"))
+    (pad 2 smd rect (at -22.5 -20.106 90) (size 0.8 0.8) (layers F.Cu F.Paste F.Mask)
+      (net 4 "Net-(AE1-Pad2)"))
+  )
   (module MultiMifare:Mifare_Chip (layer F.Cu)
     (at 157 120 270)
@@
       (net 2 "Net-(SW2-Pad1)"))
     (pad 1 smd roundrect (at -3.4 0 270) (size 1.2 5) (layers F.Cu F.Paste F.Mask) (roundrect_rratio 0.25)
-      (net 3 "Net-(AE1-Pad1)"))
+      (net 4 "Net-(AE1-Pad2)"))
   )
   (module MultiMifare:Mifare_Chip (layer F.Cu)
@@
       (net 1 "Net-(SW1-Pad1)"))
     (pad 1 smd roundrect (at -3.4 0 270) (size 1.2 5) (layers F.Cu F.Paste F.Mask) (roundrect_rratio 0.25)
-      (net 3 "Net-(AE1-Pad1)"))
+      (net 4 "Net-(AE1-Pad2)"))
   )
   (module Button_Switch_SMD:SW_SPST_TL3342 (layer F.Cu)
@@
     (fp_circle (center 0 0) (end 1 0) (layer F.Fab) (width 0.1))
     (pad 2 smd rect (at 3.15 1.9) (size 1.7 1) (layers F.Cu F.Paste F.Mask)
-      (net 4 "Net-(AE1-Pad2)"))
+      (net 3 "Net-(AE1-Pad1)"))
     (pad 2 smd rect (at -3.15 1.9) (size 1.7 1) (layers F.Cu F.Paste F.Mask)
-      (net 4 "Net-(AE1-Pad2)"))
+      (net 3 "Net-(AE1-Pad1)"))
     (pad 1 smd rect (at 3.15 -1.9) (size 1.7 1) (layers F.Cu F.Paste F.Mask)
       (net 2 "Net-(SW2-Pad1)"))
@@
     (fp_circle (center 0 0) (end 1 0) (layer F.Fab) (width 0.1))
     (pad 2 smd rect (at 3.15 1.9) (size 1.7 1) (layers F.Cu F.Paste F.Mask)
-      (net 4 "Net-(AE1-Pad2)"))
+      (net 3 "Net-(AE1-Pad1)"))
     (pad 2 smd rect (at -3.15 1.9) (size 1.7 1) (layers F.Cu F.Paste F.Mask)
-      (net 4 "Net-(AE1-Pad2)"))
+      (net 3 "Net-(AE1-Pad1)"))
     (pad 1 smd rect (at 3.15 -1.9) (size 1.7 1) (layers F.Cu F.Paste F.Mask)
       (net 1 "Net-(SW1-Pad1)"))
@@
   (gr_line (start 179.09 58.16) (end 179.09 137.4) (layer Edge.Cuts) (width 0.05))
   (gr_line (start 128.29 54.98) (end 175.91 54.98) (layer Edge.Cuts) (width 0.05))
+  (segment (start 167.85 126.55) (end 171 123.4) (width 0.762) (layer F.Cu) (net 1))
+  (segment (start 167.85 132.6) (end 167.85 126.55) (width 0.762) (layer F.Cu) (net 1))
+  (segment (start 160.15 132.6) (end 153.85 132.6) (width 0.762) (layer F.Cu) (net 2))
+  (segment (start 153.85 126.55) (end 157 123.4) (width 0.762) (layer F.Cu) (net 2))
+  (segment (start 153.85 132.6) (end 153.85 126.55) (width 0.762) (layer F.Cu) (net 2))
+  (segment (start 174.15 136.4) (end 167.85 136.4) (width 0.762) (layer F.Cu) (net 3))
+  (segment (start 167.85 136.4) (end 160.15 136.4) (width 0.762) (layer F.Cu) (net 3))
+  (segment (start 160.15 136.4) (end 153.85 136.4) (width 0.762) (layer F.Cu) (net 3))
+  (segment (start 127.29 111.452) (end 127.29 109.90651) (width 0.762) (layer F.Cu) (net 3))
+  (segment (start 152.238 136.4) (end 127.29 111.452) (width 0.762) (layer F.Cu) (net 3))
+  (segment (start 153.85 136.4) (end 152.238 136.4) (width 0.762) (layer F.Cu) (net 3))
+  (segment (start 171 116.6) (end 157 116.6) (width 0.762) (layer F.Cu) (net 4))
+  (via (at 145.9 116.6) (size 0.8) (drill 0.4) (layers F.Cu B.Cu) (net 4))
+  (segment (start 157 116.6) (end 145.9 116.6) (width 0.762) (layer F.Cu) (net 4))
+  (via (at 131.994 105.2) (size 0.8) (drill 0.4) (layers F.Cu B.Cu) (net 4))
+  (segment (start 143.394 116.6) (end 131.994 105.2) (width 0.762) (layer B.Cu) (net 4))
+  (segment (start 145.9 116.6) (end 143.394 116.6) (width 0.762) (layer B.Cu) (net 4))
 )

Commit message: DRC passed
Routing:
- net Net-(SW1-Pad1): track 10.5 -> 16.8 mm
- net Net-(AE1-Pad1): track 58.7 -> 59.3 mm
Changed lines of the file:
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@@
     (thickness 1.6)
     (drawings 8)
-    (tracks 17)
+    (tracks 21)
     (zones 0)
     (modules 5)
@@
     (mod_text_size 1 1)
     (mod_text_width 0.15)
-    (pad_size 1.524 1.524)
-    (pad_drill 0.762)
+    (pad_size 0.8 0.8)
+    (pad_drill 0)
     (pad_to_mask_clearance 0)
     (aux_axis_origin 0 0)
-    (visible_elements FFFFFF7F)
+    (visible_elements 7FFFFFFF)
     (pcbplotparams
       (layerselection 0x010fc_ffffffff)
@@
       (effects (font (size 1.524 1.524) (thickness 0.3)))
     )
-    (fp_line (start -24.83 -24.807) (end -26.43 -24.807) (layer F.Cu) (width 0.391))
-    (fp_line (start -25.2 -25.2) (end -25.2 25.2) (layer B.CrtYd) (width 0.12))
-    (fp_line (start 25.2 25.2) (end -25.2 25.2) (layer B.CrtYd) (width 0.12))
-    (fp_line (start 25.2 -25.2) (end 25.2 25.2) (layer B.CrtYd) (width 0.12))
-    (fp_line (start -25.2 -25.2) (end 25.2 -25.2) (layer B.CrtYd) (width 0.12))
     (fp_poly (pts (xy 25.005773 0.002645) (xy 25.003125 25.003125) (xy 0.002645 25.005773) (xy -24.997834 25.008421)
       (xy -24.997834 -24.235834) (xy 24.246421 -24.235834) (xy 24.243773 0.002645) (xy 24.241125 24.241125)
@@
       (xy -23.08225 23.092833) (xy 23.092833 23.092833) (xy 23.092833 -23.092834) (xy -23.84425 -23.092834)
       (xy -23.84425 23.854833) (xy 23.854833 23.854833) (xy 23.854833 -23.854834) (xy -24.60625 -23.854834)
-      (xy -24.60625 24.616833) (xy 24.616833 24.616833) (xy 24.616833 -24.616834) (xy -24.997834 -24.616834)
-      (xy -24.997834 -24.997834) (xy 25.008421 -24.997834) (xy 25.005773 0.002645)) (layer F.Cu) (width 0.01))
+      (xy -24.60625 24.616833) (xy 24.616833 24.616833) (xy 24.616833 -24.616834) (xy -26.4 -24.6095)
+      (xy -26.4 -24.9905) (xy 25.008421 -24.997834) (xy 25.005773 0.002645)) (layer F.Cu) (width 0.01))
+    (fp_line (start -25.2 -25.2) (end 25.2 -25.2) (layer B.CrtYd) (width 0.12))
+    (fp_line (start 25.2 -25.2) (end 25.2 25.2) (layer B.CrtYd) (width 0.12))
+    (fp_line (start 25.2 25.2) (end -25.2 25.2) (layer B.CrtYd) (width 0.12))
+    (fp_line (start -25.2 -25.2) (end -25.2 25.2) (layer B.CrtYd) (width 0.12))
     (pad 1 smd rect (at -26.692 -24.81 90) (size 0.8 0.8) (layers F.Cu F.Paste F.Mask)
       (net 3 "Net-(AE1-Pad1)"))
@@
   (segment (start 167.85 126.55) (end 171 123.4) (width 0.762) (layer F.Cu) (net 1))
   (segment (start 167.85 132.6) (end 167.85 126.55) (width 0.762) (layer F.Cu) (net 1))
+  (segment (start 174.15 132.6) (end 167.85 132.6) (width 0.762) (layer F.Cu) (net 1))
   (segment (start 160.15 132.6) (end 153.85 132.6) (width 0.762) (layer F.Cu) (net 2))
   (segment (start 153.85 126.55) (end 157 123.4) (width 0.762) (layer F.Cu) (net 2))
@@
   (segment (start 174.15 136.4) (end 167.85 136.4) (width 0.762) (layer F.Cu) (net 3))
   (segment (start 167.85 136.4) (end 160.15 136.4) (width 0.762) (layer F.Cu) (net 3))
+  (segment (start 153.85 136.4) (end 152.238 136.4) (width 0.762) (layer F.Cu) (net 3))
   (segment (start 160.15 136.4) (end 153.85 136.4) (width 0.762) (layer F.Cu) (net 3))
-  (segment (start 127.29 111.452) (end 127.29 109.90651) (width 0.762) (layer F.Cu) (net 3))
   (segment (start 152.238 136.4) (end 127.29 111.452) (width 0.762) (layer F.Cu) (net 3))
-  (segment (start 153.85 136.4) (end 152.238 136.4) (width 0.762) (layer F.Cu) (net 3))
+  (segment (start 127.29 111.452) (end 127.29 109.392) (width 0.762) (layer F.Cu) (net 3))
   (segment (start 171 116.6) (end 157 116.6) (width 0.762) (layer F.Cu) (net 4))
   (via (at 145.9 116.6) (size 0.8) (drill 0.4) (layers F.Cu B.Cu) (net 4))
   (segment (start 157 116.6) (end 145.9 116.6) (width 0.762) (layer F.Cu) (net 4))
+  (segment (start 143.394 116.6) (end 143.394 116.594) (width 0.762) (layer B.Cu) (net 4))
   (via (at 131.994 105.2) (size 0.8) (drill 0.4) (layers F.Cu B.Cu) (net 4))
-  (segment (start 143.394 116.6) (end 131.994 105.2) (width 0.762) (layer B.Cu) (net 4))
-  (segment (start 145.9 116.6) (end 143.394 116.6) (width 0.762) (layer B.Cu) (net 4))
+  (segment (start 132 105.2) (end 131.994 105.2) (width 0.762) (layer B.Cu) (net 4))
+  (segment (start 143.394 116.594) (end 132 105.2) (width 0.762) (layer B.Cu) (net 4))
+  (segment (start 143.4 116.6) (end 143.394 116.594) (width 0.762) (layer B.Cu) (net 4))
+  (segment (start 145.9 116.6) (end 143.4 116.6) (width 0.762) (layer B.Cu) (net 4))
 )
